File: hardware/diagnostics/diagnostics.kicad_pcb (KiCad board)
At the start: 2 copper layers, 67.8 x 45.7 mm, 9 parts, among them J1 I2C0, J2 ICSP, SW1 Input, U1 ATtiny85-20S

Commit message: Rev 1.1: - Update to latest KiCad - Fixed short in servo board - Updates to right-angle diag connector on servo boards - Fixed microproc footprint on diag board - Flipped I2C connector to top of diag board - Pass all ERC and DRC checks, add exclusions
Parts:
- added R1: 330, Resistor_SMD:R_1206_3216Metric_Pad1.30x1.75mm_HandSolder, F.Cu at (171.8, 100.6)
- J1: value I2C0 -> I2C1; moved to F.Cu
- U1: footprint Package_SO:SOIC-8_3.9x4.9mm_P1.27mm -> Package_SO:SOIC-8_5.3x5.3mm_P1.27mm
- moved J1 2.57 mm to (165.4, 77.1), turned to 180 degrees
- moved C1 1.65 mm to (171.8, 105.7)
- moved U1 0.70 mm to (165.6, 106.1)
Connections:
- net /C renamed /B
- J2 pad 2: unconnected-(J2-Pin_2-Pad2) -> Net-(J2-Pin_2)
Routing:
- net /I2C1_C: track 74.8 -> 64.2 mm, vias 1 -> 0
- net /I2C1_D: track 80.7 -> 75.3 mm, vias 1 -> 2
- net /SW: track 20.1 -> 21.9 mm
- net GND: track 3.38 -> 4.95 mm, vias 2 -> 3
- net +3.3V: track 3.03 -> 2.59 mm, vias 1 -> 0
Other:
- board text added: "ANI-DSP, Rev 1.1 Sparky Bobo Designs"
- board text added: "ICSP"
- board text added: "MISO"
- board text removed: "ANI-DSP, Rev 1.0 Sparky Bobo Designs"
- board text removed: "MISO ICSP"
